File: KiCAD Models/EOIR_gimbal/pan_centric.kicad_sch (KiCad schematic)
At the start: 11 parts

Commit message: KiCAD: update schematics — TMC2209 pinout, GPS, lens controller wiring
Co-Authored-By: Claude Sonnet 4.6 <noreply@anthropic.com>
Parts:
- added C4, C5: 100uF, symbol Device:C_Polarized
- added U23, U24: A3144, Package_TO_SOT_SMD:SOT-23W, symbol Sensor_Magnetic:A1104xLH
Connections:
- net 3V3: now also U23.1 (V_{CC}), U24.1 (V_{CC})
- net GND: now also C4.2, C5.2, U23.3 (GND), U24.3 (GND)
- net VIN+: now also C4.1, C5.1
- net E.18: now reaches U1.27 (18)
- net E.18: now also U23.2 (V_{OUT})
- net E.5: now reaches U1.28 (5)
- net E.5: now also U24.2 (V_{OUT})
- no-connect marks 29 -> 27
Other:
- note added: "FROM STATIONARY SIDE"
- note added: "PAN HALL SENSOR"
- note added: "PASS STRAIGHT THROUGH NO CONNECTION ON SHEET"
- note added: "SLIPRING REFERENCE TABLE"
- note added: "TILT HALL SENSOR"
- note added: "TO TILT SIDE"
- moved on the sheet: J3, J4, U10, U11, U4, U9
