File: KiCAD Models/EOIR_gimbal/stationary_side.kicad_sch (KiCad schematic)
At the start: 3 parts, among them J1 RJ45, J2 Conn_Coaxial_Power

Commit message: KiCAD: update schematics — TMC2209 pinout, GPS, lens controller wiring
Co-Authored-By: Claude Sonnet 4.6 <noreply@anthropic.com>
Other:
- note added: "SLIPRING REFERENCE TABLE"
Changed lines of the file:
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@@
 	(generator_version "9.0")
 	(paper "A4")
+	(text "SLIPRING REFERENCE TABLE\n"
+		(exclude_from_sim no)
+		(at 208.28 82.55 0)
+		(effects
+			(font
+				(size 1.27 1.27)
+				(italic yes)
+			)
+		)
+	)
 	(no_connect
 		(at 95.25 78.74)
@@
 				(span 1 1)
 				(fill
-					(type none)
+					(type color)
+					(color 255 0 0 1)
 				)
 				(effects
@@
 				(span 1 1)
 				(fill
-					(type none)
+					(type color)
+					(color 255 0 0 1)
+				)
+				(effects
+					(font
+						(size 1.27 1.27)
+					)
+					(justify left top)
+				)
+			)
+			(table_cell "ORANGE"
+				(exclude_from_sim no)
+				(at 189.23 88.9 0)
+				(size 20 2.54)
+				(margins 0.9525 0.9525 0.9525 0.9525)
+				(span 1 1)
+				(fill
+					(type color)
+					(color 255 0 0 1)
+				)
+				(effects
+					(font
+						(size 1.27 1.27)
+					)
+					(justify left top)
+				)
+			)
+			(table_cell "VDD+"
+				(exclude_from_sim no)
+				(at 209.23 88.9 0)
+				(size 20 2.54)
+				(margins 0.9525 0.9525 0.9525 0.9525)
+				(span 1 1)
+				(fill
+					(type color)
+					(color 255 0 0 1)
 				)
 				(effects
@@
 			(table_cell "BLACK"
 				(exclude_from_sim no)
-				(at 189.23 88.9 0)
-				(size 20 2.54)
-				(margins 0.9525 0.9525 0.9525 0.9525)
-				(span 1 1)
-				(fill
-					(type none)
+				(at 189.23 91.44 0)
+				(size 20 2.54)
+				(margins 0.9525 0.9525 0.9525 0.9525)
+				(span 1 1)
+				(fill
+					(type color)
+					(color 132 132 132 1)
 				)
 				(effects
@@
 			(table_cell "VDD-"
 				(exclude_from_sim no)
-				(at 209.23 88.9 0)
-				(size 20 2.54)
-				(margins 0.9525 0.9525 0.9525 0.9525)
-				(span 1 1)
-				(fill
-					(type none)
+				(at 209.23 91.44 0)
+				(size 20 2.54)
+				(margins 0.9525 0.9525 0.9525 0.9525)
+				(span 1 1)
+				(fill
+					(type color)
+					(color 132 132 132 1)
+				)
+				(effects
+					(font
+						(size 1.27 1.27)
+					)
+					(justify left top)
+				)
+			)
+			(table_cell "GRAY"
+				(exclude_from_sim no)
+				(at 189.23 93.98 0)
+				(size 20 2.54)
+				(margins 0.9525 0.9525 0.9525 0.9525)
+				(span 1 1)
+				(fill
+					(type color)
+					(color 132 132 132 1)
+				)
+				(effects
+					(font
+						(size 1.27 1.27)
+					)
+					(justify left top)
+				)
+			)
+			(table_cell "VDD-"
+				(exclude_from_sim no)
+				(at 209.23 93.98 0)
+				(size 20 2.54)
+				(margins 0.9525 0.9525 0.9525 0.9525)
+				(span 1 1)
+				(fill
+					(type color)
+					(color 132 132 132 1)
 				)
 				(effects
@@
 			(table_cell "WHITE"
 				(exclude_from_sim no)
-				(at 189.23 91.44 0)
+				(at 189.23 96.52 0)
 				(size 20 2.54)
 				(margins 0.9525 0.9525 0.9525 0.9525)
@@
 			(table_cell "USBD-"
 				(exclude_from_sim no)
-				(at 209.23 91.44 0)
-				(size 20 2.54)
-				(margins 0.9525 0.9525 0.9525 0.9525)
-				(span 1 1)
-				(fill
-					(type none)
-				)
-				(effects
-					(font
-						(size 1.27 1.27)
-					)
-					(justify left top)
-				)
-			)
-			(table_cell "GRAY"
-				(exclude_from_sim no)
-				(at 189.23 93.98 0)
-				(size 20 2.54)
-				(margins 0.9525 0.9525 0.9525 0.9525)
-				(span 1 1)
-				(fill
-					(type none)
-				)
-				(effects
-					(font
-						(size 1.27 1.27)
-					)
-					(justify left top)
-				)
-			)
-			(table_cell "VDD-"
-				(exclude_from_sim no)
-				(at 209.23 93.98 0)
-				(size 20 2.54)
-				(margins 0.9525 0.9525 0.9525 0.9525)
-				(span 1 1)
-				(fill
-					(type none)
-				)
-				(effects
-					(font
-						(size 1.27 1.27)
-					)
-					(justify left top)
-				)
-			)
-			(table_cell "ORANGE"
-				(exclude_from_sim no)
-				(at 189.23 96.52 0)
-				(size 20 2.54)
-				(margins 0.9525 0.9525 0.9525 0.9525)
-				(span 1 1)
-				(fill
-					(type none)
-				)
-				(effects
-					(font
-						(size 1.27 1.27)
-					)
-					(justify left top)
-				)
-			)
-			(table_cell "VDD+"
-				(exclude_from_sim no)
 				(at 209.23 96.52 0)
 				(size 20 2.54)
@@
 				(span 1 1)
 				(fill
-					(type none)
-				)
-				(effects
-					(font
-						(size 1.27 1.27)
-					)
-					(justify left top)
-				)
-			)
-			(table_cell "CAT6_RX-"
+					(type color)
+					(color 255 0 255 1)
+				)
+				(effects
+					(font
+						(size 1.27 1.27)
+					)
+					(justify left top)
+				)
+			)
+			(table_cell "CAT6_RX-/PANa1"
 				(exclude_from_sim no)
 				(at 209.23 106.68 0)
@@
 				(span 1 1)
 				(fill
-					(type none)
+					(type color)
+					(color 255 0 255 1)
 				)
 				(effects
@@
 				(span 1 1)
 				(fill
-					(type none)
-				)
-				(effects
-					(font
-						(size 1.27 1.27)
-					)
-					(justify left top)
-				)
-			)
-			(table_cell "CAT6_RX+"
+					(type color)
+					(color 255 0 255 1)
+				)
+				(effects
+					(font
+						(size 1.27 1.27)
+					)
+					(justify left top)
+				)
+			)
+			(table_cell "CAT6_RX+/PANa2"
 				(exclude_from_sim no)
 				(at 209.23 109.22 0)
@@
 				(span 1 1)
 				(fill
-					(type none)
+					(type color)
+					(color 255 0 255 1)
 				)
 				(effects
@@
 				(span 1 1)
 				(fill
-					(type none)
-				)
-				(effects
-					(font
-						(size 1.27 1.27)
-					)
-					(justify left top)
-				)
-			)
-			(table_cell "CAT6_TX-"
+					(type color)
+					(color 255 0 255 1)
+				)
+				(effects
+					(font
+						(size 1.27 1.27)
+					)
+					(justify left top)
+				)
+			)
+			(table_cell "CAT6_TX-/PANb1"
 				(exclude_from_sim no)
 				(at 209.23 111.76 0)
@@
 				(span 1 1)
 				(fill
-					(type none)
+					(type color)
+					(color 255 0 255 1)
 				)
 				(effects
@@
 				(span 1 1)
 				(fill
-					(type none)
-				)
-				(effects
-					(font
-						(size 1.27 1.27)
-					)
-					(justify left top)
-				)
-			)
-			(table_cell "CAT6_TX+"
+					(type color)
+					(color 255 0 255 1)
+				)
+				(effects
+					(font
+						(size 1.27 1.27)
+					)
+					(justify left top)
+				)
+			)
+			(table_cell "CAT6_TX+/PANb2"
 				(exclude_from_sim no)
 				(at 209.23 114.3 0)
@@
 				(span 1 1)
 				(fill
-					(type none)
+					(type color)
+					(color 255 0 255 1)
 				)
 				(effects
@@
 		(on_board yes)
 		(dnp no)
-		(fields_autoplaced yes)
 		(property "Reference" "U2"
-			(at 118.11 76.2 0)
+			(at 118.11 78.74 0)
 			(effects
 				(font
@@
 					(size 1.27 1.27)
 				)
-			)
-		)
+				(hide yes)
+			)
+		)
